File: Rev A.sch (EAGLE design)
At the start: 0 parts

Commit message: Finished schematic and PCB layout
Parts:
- added C101, C103: 1uF, rcl:C-EU150-072X183
- added C102, C104, C301, C302: 1uF, rcl:CPOL-EUE2-5
- added C105, C106: 100nF, rcl:C-EU050-025X075
- added C107, C108: 1nF, rcl:C-EU050-025X075
- added C201, C202, C203, C204: 100nF, rcl:C-EU025-025X050
- added C205, C206: 1000uF, rcl:CPOL-EUE5-10.5
- added D301, D302: BZV10, diode:BZV10
- added H201, H202, H203, H204: MOUNT-HOLE3.0, holes:MOUNT-HOLE3.0
- added IC101, IC102, IC103: LM833N, linear:LM833N
- added IC201: LM393N, linear:LM393N
- added LOWV+, LOWV-, L_IN, L_OUT, ON, PWR+, PWR-, R_IN, R_OUT, SWT_IN, SWT_OUT: (no value), adafruit:JST_2PIN-THM
- added L_BASS, L_TREBLE, L_VOL, R_BASS, R_TREBLE, R_VOL: 100kΩ, bourns:3362U
- added R101, R102, R119, R120, R121, R122: 100kΩ, rcl:R-EU_0207/10
- added R103, R104, R105, R106, R111, R112, R301, R303, R305, R307: 10kΩ, rcl:R-EU_0207/10
- added R107, R108, R109, R110: 22kΩ, rcl:R-EU_0207/10
- added R113, R114: 1MΩ, rcl:R-EU_0207/10
- added R115, R116: 1.5kΩ, rcl:R-EU_0207/10
- added R117, R118: 15kΩ, rcl:R-EU_0207/10
- added R123, R124: 1kΩ, rcl:R-EU_0207/10
- added R201, R304, R308: 4.7kΩ, rcl:R-EU_0207/10
- added R302, R306: 27kΩ, rcl:R-EU_0207/10
Connections:
- new net GND: C205.+, C206.-, C301.-, C302.+, D301.A, D302.C, L_IN.1, L_OUT.1, L_TREBLE.1, L_VOL.1, PWR+.1, PWR-.2, R101.1, R102.1, R103.1, R104.1, R108.1, R110.1, R113.1, R114.1, R117.1, R118.1, R119.1, R120.1, R303.1, R307.1, R_IN.1, R_OUT.1, R_TREBLE.1, R_VOL.1
- new net N$1: L_OUT.2, R124.2
- new net N$10: IC201B.-IN, R306.2, R307.2
- new net N$11: IC201A.OUT, R304.1
- new net N$12: LOWV-.1, R308.2
- new net N$13: IC201B.OUT, R308.1
- new net N$2: R123.2, R_OUT.2
- new net N$22: C103.1, C104.+, L_IN.2
- new net N$3: C301.+, D301.C, IC201A.-IN, R301.1
- new net N$4: C101.2, C102.-, IC101A.+IN, R101.2
- new net N$5: C302.-, D302.A, IC201B.+IN, R305.1
- new net N$55: ON.1, R201.2
- new net N$56: IC102A.-IN, IC102A.OUT, R115.1
- new net N$57: C105.2, R107.1, R_BASS.3
- new net N$58: IC103A.+IN, R117.2, R_VOL.2
- new net N$59: IC101A.-IN, R103.2, R105.1
- new net N$6: LOWV+.1, R304.2
- new net N$60: R115.2, R_VOL.3
- new net N$61: C105.1, R108.2, R_BASS.1
- new net N$62: IC103A.-IN, R119.2, R121.1
- new net N$63: IC103A.OUT, R121.2, R123.1
- new net N$64: R111.1, R_BASS.2
- new net N$65: C107.1, IC102A.+IN, R111.2, R113.2
- new net N$66: C107.2, R_TREBLE.2
- new net N$67: IC102B.-IN, IC102B.OUT, R116.1
- new net N$68: IC101B.-IN, R104.2, R106.1
- new net N$69: IC101A.OUT, R105.2, R107.2, R_TREBLE.3
- new net N$7: C103.2, C104.-, IC101B.+IN, R102.2
- new net N$70: IC103B.+IN, L_VOL.2, R118.2
- new net N$71: L_VOL.3, R116.2
- new net N$72: C106.2, L_BASS.3, R109.1
- new net N$73: C106.1, L_BASS.1, R110.2
- new net N$74: L_BASS.2, R112.1
- new net N$75: C108.1, IC102B.+IN, R112.2, R114.2
- new net N$76: C108.2, L_TREBLE.2
- new net N$77: IC101B.OUT, L_TREBLE.3, R106.2, R109.2
- new net N$78: IC103B.-IN, R120.2, R122.1
- new net N$79: IC103B.OUT, R122.2, R124.1
- new net N$8: C101.1, C102.+, R_IN.2
- new net N$9: IC201A.+IN, R302.2, R303.2
- new net SWTIN+: PWR+.2, SWT_IN.2
- new net SWTIN-: PWR-.1, SWT_IN.1
- new net V+: C201.1, C202.1, C203.1, C204.1, C206.+, IC101P.V+, IC102P.V+, IC103P.V+, IC201P.V+, LOWV+.2, LOWV-.2, ON.2, R301.2, R302.1, SWT_OUT.2
- new net V-: C201.2, C202.2, C203.2, C204.2, C205.-, IC101P.V-, IC102P.V-, IC103P.V-, IC201P.V-, R201.1, R305.2, R306.1, SWT_OUT.1
Other:
- note added: "+2.0V"
- note added: "-2.0V"
- note added: "1n5226 3.3V Zener"
